Commit message: update joint limits

File: soarm100_description/urdf/soarm100_5dof.ros2control.xacro (robot description, xacro)
@@ -29,6 +29,6 @@
       <joint name="wrist_pitch_joint">
          <command_interface name="position">
-            <param name="min">-${PI/2}</param>
-            <param name="max">${PI/2}</param>
+            <param name="min">-${PI}</param>
+            <param name="max">${PI/4}</param>
          </command_interface>
          <state_interface name="position"></state_interface>
@@ -43,6 +43,6 @@
       <joint name="jaw_joint">
          <command_interface name="position">
-            <param name="min">-${PI/2}</param>
-            <param name="max">${PI/2}</param>
+            <param name="min">-${PI/18}</param>
+            <param name="max">${PI/3}</param>
          </command_interface>
          <state_interface name="position"></state_interface>

File: soarm100_description/urdf/soarm100_5dof_base.urdf.xacro (robot description, xacro)
@@ -194,5 +194,5 @@
         <child link="wrist_link" />
         <axis xyz="1 0 0" />
-        <limit lower="-${PI/2}" upper="${PI/2}" effort="${effort}" velocity="${velocity}"/>
+        <limit lower="-${PI}" upper="${PI/4}" effort="${effort}" velocity="${velocity}"/>
     </joint>
     <link name="fixed_jaw_link">
@@ -268,5 +268,5 @@
         <child link="moving_jaw_link" />
         <axis xyz="0 0 1" />
-        <limit lower="-${PI/2}" upper="${PI/2}" effort="${effort}" velocity="${velocity}"/>
+        <limit lower="-${PI/18}" upper="${PI/3}" effort="${effort}" velocity="${velocity}"/>
     </joint>
 </robot>
